Commit message: gazebo_additions.xacro
новая физика

File: ros2_ws/src/my_robot_gazebo/urdf/my_robot.urdf.xacro (robot description, xacro)
@@ -1,129 +1,28 @@
 <?xml version="1.0"?>
-<robot name="my_robot" xmlns:xacro="http://www.ros.org/wiki/xacro">
-  <xacro:property name="base_length" value="0.30"/>
-  <xacro:property name="base_width"  value="0.20"/>
-  <xacro:property name="base_height" value="0.10"/>
-  <xacro:property name="base_mass"   value="2.0"/>
-  <xacro:property name="wheel_radius"    value="0.05"/>
-  <xacro:property name="wheel_length"    value="0.04"/>
-  <xacro:property name="wheel_mass"      value="0.2"/>
-  <xacro:property name="wheel_separation" value="0.24"/>
-  <xacro:property name="caster_radius" value="0.025"/>
-  <xacro:property name="caster_mass"   value="0.05"/>
-  <xacro:macro name="box_inertia" params="m x y z">
-    <inertial>
-      <mass value="${m}"/>
-      <inertia
-        ixx="${m*(y*y + z*z)/12}" ixy="0.0" ixz="0.0"
-        iyy="${m*(x*x + z*z)/12}" iyz="0.0"
-        izz="${m*(x*x + y*y)/12}"/>
-    </inertial>
-  </xacro:macro>
-  <xacro:macro name="cylinder_inertia" params="m r l">
-    <inertial>
-      <mass value="${m}"/>
-      <inertia
-        ixx="${m*(3*r*r + l*l)/12}" ixy="0.0" ixz="0.0"
-        iyy="${m*(3*r*r + l*l)/12}" iyz="0.0"
-        izz="${m*r*r/2}"/>
-    </inertial>
-  </xacro:macro>
-  <xacro:macro name="sphere_inertia" params="m r">
-    <inertial>
-      <mass value="${m}"/>
-      <inertia
-        ixx="${2*m*r*r/5}" ixy="0.0" ixz="0.0"
-        iyy="${2*m*r*r/5}" iyz="0.0"
-        izz="${2*m*r*r/5}"/>
-    </inertial>
-  </xacro:macro>
+<robot xmlns:xacro="http://www.ros.org/wiki/xacro" name="r2d2_gazebo_wrapper">
+  <xacro:include filename="$(find my_robot_gazebo)/urdf/05-visual.urdf" />
   <link name="base_footprint"/>
-  <link name="base_link">
-    <visual>
-      <geometry><box size="${base_length} ${base_width} ${base_height}"/></geometry>
-      <material name="blue"><color rgba="0.2 0.4 0.9 1.0"/></material>
-    </visual>
-    <collision>
-      <geometry><box size="${base_length} ${base_width} ${base_height}"/></geometry>
-    </collision>
-    <xacro:box_inertia m="${base_mass}" x="${base_length}" y="${base_width}" z="${base_height}"/>
-  </link>
   <joint name="base_footprint_to_base" type="fixed">
     <parent link="base_footprint"/>
     <child link="base_link"/>
-    <origin xyz="0 0 ${wheel_radius}" rpy="0 0 0"/>
+    <origin xyz="0 0 0" rpy="0 0 0"/>
   </joint>
-  <xacro:macro name="wheel" params="prefix y_offset">
-    <link name="${prefix}_wheel_link">
-      <visual>
-        <origin xyz="0 0 0" rpy="${pi/2} 0 0"/>
-        <geometry><cylinder radius="${wheel_radius}" length="${wheel_length}"/></geometry>
-        <material name="black"><color rgba="0.1 0.1 0.1 1.0"/></material>
-      </visual>
-      <collision>
-        <origin xyz="0 0 0" rpy="${pi/2} 0 0"/>
-        <geometry><cylinder radius="${wheel_radius}" length="${wheel_length}"/></geometry>
-      </collision>
-      <xacro:cylinder_inertia m="${wheel_mass}" r="${wheel_radius}" l="${wheel_length}"/>
-    </link>
-    <joint name="${prefix}_wheel_joint" type="continuous">
-      <parent link="base_link"/>
-      <child link="${prefix}_wheel_link"/>
-      <origin xyz="0 ${y_offset} ${-base_height/2}" rpy="0 0 0"/>
-      <axis xyz="0 1 0"/>
-    </joint>
-  </xacro:macro>
-  <xacro:wheel prefix="left"  y_offset="${ wheel_separation/2}"/>
-  <xacro:wheel prefix="right" y_offset="${-wheel_separation/2}"/>
-  <link name="caster_link">
-    <visual>
-      <geometry><sphere radius="${caster_radius}"/></geometry>
-      <material name="gray"><color rgba="0.5 0.5 0.5 1.0"/></material>
-    </visual>
+  <gazebo reference="base_link">
     <collision>
-      <geometry><sphere radius="${caster_radius}"/></geometry>
+      <geometry>
+        <cylinder length="0.6" radius="0.2"/>
+      </geometry>
     </collision>
-    <xacro:sphere_inertia m="${caster_mass}" r="${caster_radius}"/>
-  </link>
-  <joint name="caster_joint" type="fixed">
-    <parent link="base_link"/>
-    <child link="caster_link"/>
-    <origin xyz="${base_length/2 - 0.03} 0 ${-base_height/2 - (wheel_radius - caster_radius)}" rpy="0 0 0"/>
-  </joint>
-  <link name="lidar_link">
-    <visual>
-      <geometry><cylinder radius="0.04" length="0.04"/></geometry>
-      <material name="red"><color rgba="0.9 0.1 0.1 1.0"/></material>
-    </visual>
-    <collision>
-      <geometry><cylinder radius="0.04" length="0.04"/></geometry>
-    </collision>
-    <xacro:cylinder_inertia m="0.1" r="0.04" l="0.04"/>
-  </link>
-  <joint name="lidar_joint" type="fixed">
-    <parent link="base_link"/>
-    <child link="lidar_link"/>
-    <origin xyz="0.05 0 ${base_height/2 + 0.02}" rpy="0 0 0"/>
-  </joint>
-  <link name="imu_link">
-    <visual>
-      <geometry><box size="0.03 0.03 0.01"/></geometry>
-      <material name="green"><color rgba="0.1 0.8 0.1 1.0"/></material>
-    </visual>
-    <xacro:box_inertia m="0.01" x="0.03" y="0.03" z="0.01"/>
-  </link>
-  <joint name="imu_joint" type="fixed">
-    <parent link="base_link"/>
-    <child link="imu_link"/>
-    <origin xyz="0 0 ${base_height/2 + 0.005}" rpy="0 0 0"/>
-  </joint>
-  <!-- ============================ Gazebo Harmonic plugins ============================ -->
+    <inertial>
+      <mass value="10.0"/>
+      <inertia ixx="0.4" ixy="0.0" ixz="0.0" iyy="0.4" iyz="0.0" izz="0.2"/>
+    </inertial>
+  </gazebo>
   <gazebo>
-    <plugin filename="gz-sim-diff-drive-system"
-            name="gz::sim::systems::DiffDrive">
-      <left_joint>left_wheel_joint</left_joint>
-      <right_joint>right_wheel_joint</right_joint>
-      <wheel_separation>${wheel_separation}</wheel_separation>
-      <wheel_radius>${wheel_radius}</wheel_radius>
+    <plugin filename="gz-sim-diff-drive-system" name="gz::sim::systems::DiffDrive">
+      <left_joint>left_front_wheel_joint</left_joint>
+      <right_joint>right_front_wheel_joint</right_joint>
+      <wheel_separation>0.44</wheel_separation>
+      <wheel_radius>0.035</wheel_radius>
       <odom_publish_frequency>30</odom_publish_frequency>
       <topic>cmd_vel</topic>
@@ -132,46 +31,14 @@
       <frame_id>odom</frame_id>
       <child_frame_id>base_footprint</child_frame_id>
-      <max_linear_acceleration>2.0</max_linear_acceleration>
-      <max_angular_acceleration>3.0</max_angular_acceleration>
-    </plugin>
-    <plugin filename="gz-sim-joint-state-publisher-system"
-            name="gz::sim::systems::JointStatePublisher">
-      <topic>joint_states</topic>
-      <joint_name>left_wheel_joint</joint_name>
-      <joint_name>right_wheel_joint</joint_name>
     </plugin>
   </gazebo>
-  <gazebo reference="lidar_link">
-    <sensor name="lidar" type="gpu_lidar">
-      <pose>0 0 0 0 0 0</pose>
-      <topic>scan</topic>
-      <gz_frame_id>lidar_link</gz_frame_id>
-      <update_rate>10</update_rate>
-      <ray>
-        <scan>
-          <horizontal>
-            <samples>360</samples>
-            <resolution>1</resolution>
-            <min_angle>-3.14159</min_angle>
-            <max_angle>3.14159</max_angle>
-          </horizontal>
-        </scan>
-        <range>
-          <min>0.12</min>
-          <max>8.0</max>
-          <resolution>0.01</resolution>
-        </range>
-      </ray>
-      <always_on>1</always_on>
-      <visualize>true</visualize>
-    </sensor>
-  </gazebo>
-  <gazebo reference="imu_link">
-    <sensor name="imu" type="imu">
-      <topic>imu</topic>
-      <gz_frame_id>imu_link</gz_frame_id>
-      <update_rate>100</update_rate>
-      <always_on>1</always_on>
-    </sensor>
+  <gazebo>
+    <plugin filename="gz-sim-joint-state-publisher-system" name="gz::sim::systems::JointStatePublisher">
+      <topic>joint_states</topic>
+      <joint_name>left_front_wheel_joint</joint_name>
+      <joint_name>left_back_wheel_joint</joint_name>
+      <joint_name>right_front_wheel_joint</joint_name>
+      <joint_name>right_back_wheel_joint</joint_name>
+    </plugin>
   </gazebo>
 </robot>

Commit message: Update my_robot.urdf.xacro
я не буду это комментировать

File: ros2_ws/src/my_robot_gazebo/urdf/my_robot.urdf.xacro (robot description, xacro)
@@ -1,22 +1,5 @@
 <?xml version="1.0"?>
-<robot xmlns:xacro="http://www.ros.org/wiki/xacro" name="r2d2_gazebo_wrapper">
+<robot xmlns:xacro="http://www.ros.org/wiki/xacro" name="r2d2_gazebo">
   <xacro:include filename="$(find my_robot_gazebo)/urdf/05-visual.urdf" />
-  <link name="base_footprint"/>
-  <joint name="base_footprint_to_base" type="fixed">
-    <parent link="base_footprint"/>
-    <child link="base_link"/>
-    <origin xyz="0 0 0" rpy="0 0 0"/>
-  </joint>
-  <gazebo reference="base_link">
-    <collision>
-      <geometry>
-        <cylinder length="0.6" radius="0.2"/>
-      </geometry>
-    </collision>
-    <inertial>
-      <mass value="10.0"/>
-      <inertia ixx="0.4" ixy="0.0" ixz="0.0" iyy="0.4" iyz="0.0" izz="0.2"/>
-    </inertial>
-  </gazebo>
   <gazebo>
     <plugin filename="gz-sim-diff-drive-system" name="gz::sim::systems::DiffDrive">
@@ -30,5 +13,5 @@
       <tf_topic>tf</tf_topic>
       <frame_id>odom</frame_id>
-      <child_frame_id>base_footprint</child_frame_id>
+      <child_frame_id>base_link</child_frame_id>
     </plugin>
   </gazebo>

Commit message: chore: Sanyok review (#2)
* Update first_world.md

теперь мир запускается отдельно

* diff-drive.md

изменены имена суставов и размеры робота

* join state publisher.md

добавлены колеса 😆

* gazebo_additions.xacro

новая физика

* lesson5.md

добавлена физика к модели робота из пятого урока

* Update my_robot.urdf.xacro

я не буду это комментировать

* !

* !

* !

* Add files via upload

* Update 02-first-world.md

* Update 03-urdf-xacro.md

* Update 03-urdf-xacro.md

* Update 03-urdf-xacro.md

* Create cylinder_orientation.svg

* Update cylinder_orientation.svg

* Update 04-spawn-robot.md

* Update 05-bridge.md

* Create rviz_lidar.png

* Update 06-sensors.md

* Update 07-world-teleop.md

* Update 07-world-teleop.md

* Update 08-balancer.md

* Add files via upload

* Delete lesson 8 (Gazebo)/first_world.md

* Delete lesson 8 (Gazebo)/custom_world_teleop.md

* Delete lesson 8 (Gazebo)/installing_gazebo.md

* Delete lesson 8 (Gazebo)/ros_gz_bridge.md

* Delete lesson 8 (Gazebo)/sensors_lidar_imu.md

* Delete lesson 8 (Gazebo)/spawning_urdf.md

* Delete lesson 8 (Gazebo)/lqr_theory.docx

* Add files via upload

* Update 08-balancer.md

* Delete lesson 8 (Gazebo)/images/rviz_lidar.png

* Update 08-balancer.md

* Update 06-sensors.md

* Update 06-sensors.md

* Update 05-bridge.md

---------

Co-authored-by: m2311021 <145960653+m2311021@users.noreply.github.com>

File: ros2_ws/src/my_robot_gazebo/urdf/my_robot.urdf.xacro (robot description, xacro)
@@ -1,129 +1,11 @@
 <?xml version="1.0"?>
-<robot name="my_robot" xmlns:xacro="http://www.ros.org/wiki/xacro">
-  <xacro:property name="base_length" value="0.30"/>
-  <xacro:property name="base_width"  value="0.20"/>
-  <xacro:property name="base_height" value="0.10"/>
-  <xacro:property name="base_mass"   value="2.0"/>
-  <xacro:property name="wheel_radius"    value="0.05"/>
-  <xacro:property name="wheel_length"    value="0.04"/>
-  <xacro:property name="wheel_mass"      value="0.2"/>
-  <xacro:property name="wheel_separation" value="0.24"/>
-  <xacro:property name="caster_radius" value="0.025"/>
-  <xacro:property name="caster_mass"   value="0.05"/>
-  <xacro:macro name="box_inertia" params="m x y z">
-    <inertial>
-      <mass value="${m}"/>
-      <inertia
-        ixx="${m*(y*y + z*z)/12}" ixy="0.0" ixz="0.0"
-        iyy="${m*(x*x + z*z)/12}" iyz="0.0"
-        izz="${m*(x*x + y*y)/12}"/>
-    </inertial>
-  </xacro:macro>
-  <xacro:macro name="cylinder_inertia" params="m r l">
-    <inertial>
-      <mass value="${m}"/>
-      <inertia
-        ixx="${m*(3*r*r + l*l)/12}" ixy="0.0" ixz="0.0"
-        iyy="${m*(3*r*r + l*l)/12}" iyz="0.0"
-        izz="${m*r*r/2}"/>
-    </inertial>
-  </xacro:macro>
-  <xacro:macro name="sphere_inertia" params="m r">
-    <inertial>
-      <mass value="${m}"/>
-      <inertia
-        ixx="${2*m*r*r/5}" ixy="0.0" ixz="0.0"
-        iyy="${2*m*r*r/5}" iyz="0.0"
-        izz="${2*m*r*r/5}"/>
-    </inertial>
-  </xacro:macro>
-  <link name="base_footprint"/>
-  <link name="base_link">
-    <visual>
-      <geometry><box size="${base_length} ${base_width} ${base_height}"/></geometry>
-      <material name="blue"><color rgba="0.2 0.4 0.9 1.0"/></material>
-    </visual>
-    <collision>
-      <geometry><box size="${base_length} ${base_width} ${base_height}"/></geometry>
-    </collision>
-    <xacro:box_inertia m="${base_mass}" x="${base_length}" y="${base_width}" z="${base_height}"/>
-  </link>
-  <joint name="base_footprint_to_base" type="fixed">
-    <parent link="base_footprint"/>
-    <child link="base_link"/>
-    <origin xyz="0 0 ${wheel_radius}" rpy="0 0 0"/>
-  </joint>
-  <xacro:macro name="wheel" params="prefix y_offset">
-    <link name="${prefix}_wheel_link">
-      <visual>
-        <origin xyz="0 0 0" rpy="${pi/2} 0 0"/>
-        <geometry><cylinder radius="${wheel_radius}" length="${wheel_length}"/></geometry>
-        <material name="black"><color rgba="0.1 0.1 0.1 1.0"/></material>
-      </visual>
-      <collision>
-        <origin xyz="0 0 0" rpy="${pi/2} 0 0"/>
-        <geometry><cylinder radius="${wheel_radius}" length="${wheel_length}"/></geometry>
-      </collision>
-      <xacro:cylinder_inertia m="${wheel_mass}" r="${wheel_radius}" l="${wheel_length}"/>
-    </link>
-    <joint name="${prefix}_wheel_joint" type="continuous">
-      <parent link="base_link"/>
-      <child link="${prefix}_wheel_link"/>
-      <origin xyz="0 ${y_offset} ${-base_height/2}" rpy="0 0 0"/>
-      <axis xyz="0 1 0"/>
-    </joint>
-  </xacro:macro>
-  <xacro:wheel prefix="left"  y_offset="${ wheel_separation/2}"/>
-  <xacro:wheel prefix="right" y_offset="${-wheel_separation/2}"/>
-  <link name="caster_link">
-    <visual>
-      <geometry><sphere radius="${caster_radius}"/></geometry>
-      <material name="gray"><color rgba="0.5 0.5 0.5 1.0"/></material>
-    </visual>
-    <collision>
-      <geometry><sphere radius="${caster_radius}"/></geometry>
-    </collision>
-    <xacro:sphere_inertia m="${caster_mass}" r="${caster_radius}"/>
-  </link>
-  <joint name="caster_joint" type="fixed">
-    <parent link="base_link"/>
-    <child link="caster_link"/>
-    <origin xyz="${base_length/2 - 0.03} 0 ${-base_height/2 - (wheel_radius - caster_radius)}" rpy="0 0 0"/>
-  </joint>
-  <link name="lidar_link">
-    <visual>
-      <geometry><cylinder radius="0.04" length="0.04"/></geometry>
-      <material name="red"><color rgba="0.9 0.1 0.1 1.0"/></material>
-    </visual>
-    <collision>
-      <geometry><cylinder radius="0.04" length="0.04"/></geometry>
-    </collision>
-    <xacro:cylinder_inertia m="0.1" r="0.04" l="0.04"/>
-  </link>
-  <joint name="lidar_joint" type="fixed">
-    <parent link="base_link"/>
-    <child link="lidar_link"/>
-    <origin xyz="0.05 0 ${base_height/2 + 0.02}" rpy="0 0 0"/>
-  </joint>
-  <link name="imu_link">
-    <visual>
-      <geometry><box size="0.03 0.03 0.01"/></geometry>
-      <material name="green"><color rgba="0.1 0.8 0.1 1.0"/></material>
-    </visual>
-    <xacro:box_inertia m="0.01" x="0.03" y="0.03" z="0.01"/>
-  </link>
-  <joint name="imu_joint" type="fixed">
-    <parent link="base_link"/>
-    <child link="imu_link"/>
-    <origin xyz="0 0 ${base_height/2 + 0.005}" rpy="0 0 0"/>
-  </joint>
-  <!-- ============================ Gazebo Harmonic plugins ============================ -->
+<robot xmlns:xacro="http://www.ros.org/wiki/xacro" name="r2d2_gazebo">
+  <xacro:include filename="$(find my_robot_gazebo)/urdf/05-visual.urdf" />
   <gazebo>
-    <plugin filename="gz-sim-diff-drive-system"
-            name="gz::sim::systems::DiffDrive">
-      <left_joint>left_wheel_joint</left_joint>
-      <right_joint>right_wheel_joint</right_joint>
-      <wheel_separation>${wheel_separation}</wheel_separation>
-      <wheel_radius>${wheel_radius}</wheel_radius>
+    <plugin filename="gz-sim-diff-drive-system" name="gz::sim::systems::DiffDrive">
+      <left_joint>left_front_wheel_joint</left_joint>
+      <right_joint>right_front_wheel_joint</right_joint>
+      <wheel_separation>0.44</wheel_separation>
+      <wheel_radius>0.035</wheel_radius>
       <odom_publish_frequency>30</odom_publish_frequency>
       <topic>cmd_vel</topic>
@@ -131,47 +13,15 @@
       <tf_topic>tf</tf_topic>
       <frame_id>odom</frame_id>
-      <child_frame_id>base_footprint</child_frame_id>
-      <max_linear_acceleration>2.0</max_linear_acceleration>
-      <max_angular_acceleration>3.0</max_angular_acceleration>
-    </plugin>
-    <plugin filename="gz-sim-joint-state-publisher-system"
-            name="gz::sim::systems::JointStatePublisher">
-      <topic>joint_states</topic>
-      <joint_name>left_wheel_joint</joint_name>
-      <joint_name>right_wheel_joint</joint_name>
+      <child_frame_id>base_link</child_frame_id>
     </plugin>
   </gazebo>
-  <gazebo reference="lidar_link">
-    <sensor name="lidar" type="gpu_lidar">
-      <pose>0 0 0 0 0 0</pose>
-      <topic>scan</topic>
-      <gz_frame_id>lidar_link</gz_frame_id>
-      <update_rate>10</update_rate>
-      <ray>
-        <scan>
-          <horizontal>
-            <samples>360</samples>
-            <resolution>1</resolution>
-            <min_angle>-3.14159</min_angle>
-            <max_angle>3.14159</max_angle>
-          </horizontal>
-        </scan>
-        <range>
-          <min>0.12</min>
-          <max>8.0</max>
-          <resolution>0.01</resolution>
-        </range>
-      </ray>
-      <always_on>1</always_on>
-      <visualize>true</visualize>
-    </sensor>
-  </gazebo>
-  <gazebo reference="imu_link">
-    <sensor name="imu" type="imu">
-      <topic>imu</topic>
-      <gz_frame_id>imu_link</gz_frame_id>
-      <update_rate>100</update_rate>
-      <always_on>1</always_on>
-    </sensor>
+  <gazebo>
+    <plugin filename="gz-sim-joint-state-publisher-system" name="gz::sim::systems::JointStatePublisher">
+      <topic>joint_states</topic>
+      <joint_name>left_front_wheel_joint</joint_name>
+      <joint_name>left_back_wheel_joint</joint_name>
+      <joint_name>right_front_wheel_joint</joint_name>
+      <joint_name>right_back_wheel_joint</joint_name>
+    </plugin>
   </gazebo>
 </robot>
